Commit message: Updated Scripts

File: src/align_description/urdf/align.urdf.xacro (robot description, xacro)
@@ -270,5 +270,5 @@
   </joint>
   <joint name="hokuyo_joint" type="fixed">
-    <origin xyz="1.1 0.00 0.1" rpy="0 0 0" />
+    <origin xyz="1 0.00 0.1" rpy="0 0 0" />
     <parent link="base_link" />
     <child link="hokuyo" />
@@ -303,5 +303,5 @@
   </link>
  <joint name="camera_joint" type="fixed">
-    <origin xyz="1.1 0 0.2" rpy="0 0 0"/>
+    <origin xyz="1 0 0.2" rpy="0 0 0"/>
     <parent link="base_link"/>
     <child link="camera_link"/>
@@ -312,5 +312,5 @@
       <origin xyz="0 0 0" rpy="0 0 0"/>
       <geometry>
-    <box size="0.1 0.1 0.1"/>
+    <box size="0.01 0.01 0.01"/>
       </geometry>
     </collision>
@@ -435,6 +435,6 @@
             <samples>560</samples>
             <resolution>1</resolution>
-            <min_angle>-1.22173</min_angle>
-            <max_angle>1.22173</max_angle>
+            <min_angle>-1.221730476396</min_angle>
+            <max_angle>1.221730476396</max_angle>
           </horizontal>
         </scan>
@@ -547,5 +547,5 @@
   </gazebo>
   <xacro:include filename="$(find velodyne_description)/urdf/VLP-16.urdf.xacro"/>
-  <VLP-16 parent = "base_link" name="/velodyne" topic="/velodyne_points" hz="10" samples="440/">
+  <VLP-16 parent = "base_link" name="/velodyne" topic="/velodyne_points" hz="1" samples="440" max_range="20">
     <origin xyz="0 0 0.5" rpy="0 0 0"/>
   </VLP-16>

Commit message: Added Retracing Script

File: src/align_description/urdf/align.urdf.xacro (robot description, xacro)
@@ -25,5 +25,5 @@
        vertical wheel travel. -->
   <xacro:property name="wheelbase" value="1.9"/>
-  <xacro:property name="hex_hub_dist" value="1.45"/>
+  <xacro:property name="hex_hub_dist" value="1.36"/>
   <xacro:property name="axle_length" value="0.03"/>
   <xacro:property name="wheel_travel" value="0.084"/>
@@ -270,5 +270,5 @@
   </joint>
   <joint name="hokuyo_joint" type="fixed">
-    <origin xyz="1 0.00 0.1" rpy="0 0 0" />
+    <origin xyz="1.1 0.00 0.1" rpy="0 0 0" />
     <parent link="base_link" />
     <child link="hokuyo" />
@@ -303,5 +303,5 @@
   </link>
  <joint name="camera_joint" type="fixed">
-    <origin xyz="1 0 0.2" rpy="0 0 0"/>
+    <origin xyz="1.1 0 0.2" rpy="0 0 0"/>
     <parent link="base_link"/>
     <child link="camera_link"/>

Commit message: Changed HMS Logs

File: src/align_description/urdf/align.urdf.xacro (robot description, xacro)
@@ -248,5 +248,5 @@
 <link name="lift_link">
     <visual>
-      <origin rpy="0 0 1.57079633" xyz="0 0 0"/>
+      <origin rpy="0 0 1.57079633" xyz="-0.02 0 0"/>
       <geometry>
         <mesh filename="package://align_description/meshes/lift_f.dae"/>

Commit message: Ported Goal Publisher to Autoware simulation, added lift

File: src/align_description/urdf/align.urdf.xacro (robot description, xacro)
@@ -246,4 +246,10 @@
     <material>Gazebo/Grey</material>
   </gazebo> -->
+ <joint name="base_link_to_lift" type="prismatic">
+    <parent link="base_link"/>
+    <child link="lift_link"/>
+    <axis xyz="0 0 1"/>
+    <limit lower="0" upper="3" effort="1000" velocity="0.2"/>
+  </joint>
 <link name="lift_link">
     <visual>
@@ -254,10 +260,20 @@
       <material name="chassis_mat"/>
     </visual>
-    <!-- <collision>
-      <origin rpy="0 0 1.57079633" xyz="0 0 0"/>
-      <geometry>
-        <mesh filename="package://align_description/meshes/chassis.stl" scale="0.001 0.001 0.001"/>
-      </geometry>
-    </collision> -->
+    <!-- CAN VBE MULTIPLE COLLISIONS -->
+    <collision>
+      <origin rpy="0 0 1.57079633" xyz="0 0 0.55"/>
+      <geometry>
+        <box size="0.5 0.5 0.01"/>
+        <!-- <mesh filename="package://align_description/meshes/chassis.stl" scale="0.001 0.001 0.001"/> -->
+      </geometry>
+    </collision>
+    <inertial>
+        <origin rpy="0 0 1.57079633" xyz="-0.02 0 0"/>
+        <mass value="1"/>
+        <inertia
+          ixx="1.0" ixy="0.0" ixz="0.0"
+          iyy="1.0" iyz="0.0"
+          izz="1.0"/>
+    </inertial>
   </link>
   <gazebo reference="lift_link">
@@ -265,8 +281,4 @@
     <selfCollide>false</selfCollide>
   </gazebo>
- <joint name="base_link_to_lift" type="fixed">
-    <parent link="base_link"/>
-    <child link="lift_link"/>
-  </joint>
   <joint name="hokuyo_joint" type="fixed">
     <origin xyz="1.1 0.00 0.1" rpy="0 0 0" />
@@ -550,3 +562,13 @@
     <origin xyz="0 0 0.5" rpy="0 0 0"/>
   </VLP-16>
+   <transmission name="lift_transmission">
+    <type>transmission_interface/SimpleTransmission</type>
+    <joint name="base_link_to_lift">
+      <hardwareInterface>hardware_interface/VelocityJointInterface</hardwareInterface>
+    </joint>
+    <actuator name="lift_motor">
+      <hardwareInterface>hardware_interface/VelocityJointInterface</hardwareInterface>
+      <mechanicalReduction>1</mechanicalReduction>
+    </actuator>
+  </transmission>
 </robot>
